File: DC-DC 12-450V.kicad_sch (KiCad schematic)
At the start: 31 parts, among them J1 12V input, J2 HV output, Q1 IRF3205, Q2 S8050, U1 UC3843BN_DIP8

Commit message: Add files via upload
Parts:
- added D4: PESD12VL1BA, Diode_SMD:D_SOD-323, symbol Diode:SD12_SOD323
- added F2: 1.5A/13.2V, Fuse:Fuse_1206_3216Metric_Pad1.42x1.75mm_HandSolder, symbol Device:Polyfuse_Small
Connections:
- net +12V: now also F2.1; no longer C8.1, Q2.3 (C), U1.7 (VCC)
- net GND: now also D4.2 (A2)
- new net VCC: C8.1, D4.1 (A1), F2.2, Q2.3 (C), U1.7 (VCC)
