File: DC-DC 12-450V.kicad_pcb (KiCad board)
At the start: 2 copper layers, 85 x 50 mm, 44 parts, among them J1 12V input, J2 HV output, Q1 IRF3205, Q2 S8050, U1 UC3843BN_DIP8

Commit message: Add files via upload
Parts:
- added D4: PESD12VL1BA, Diode_SMD:D_SOD-323, F.Cu at (126.8, 80.0)
- added F2: 1.5A/13.2V, Fuse:Fuse_1206_3216Metric_Pad1.42x1.75mm_HandSolder, F.Cu at (129.5, 85.5)
- R11: value 0.015R -> 0.015R/3W
- moved C8 4.01 mm to (126.8, 76.0)
- moved R7 1.44 mm to (125.5, 91.2), turned to 0 degrees
Connections:
- C8 pad 1: +12V -> /VCC
- Q2 pad 1: Net-(Q2-B) -> unconnected-(Q2-B-Pad1)
- Q2 pad 3: +12V -> /VCC
- R10 pad 1: Net-(Q2-B) -> Net-(R10-Pad1)
- RV1 pad 2: Net-(Q2-B) -> Net-(R10-Pad1)
- RV1 pad 3: Net-(Q2-B) -> Net-(R10-Pad1)
- U1 pad 7: +12V -> /VCC
Routing:
- net +12V: track 108.3 -> 73.2 mm
- net /VCC: track 0.00 -> 34.5 mm
- net Net-(Q2-B): track 14.7 -> 0.00 mm
- net (no net): track 0.00 -> 14.7 mm
- net Net-(U1-OUT): track 5.66 -> 6.62 mm
- net Net-(Q1-G): vias 2 -> 4

Commit message: Add files via upload
Routing:
- net GND: track 144.0 -> 144.3 mm, vias 21 -> 48
- net Net-(U1-CS): vias 2 -> 3
